Commit message: Add files via upload

File: description/urdf/description.urdf (robot description, URDF)
Before this commit: robot description, 9 links, 8 joints
Links:
- link base_link: mass 9.56039071848755 -> 5.36255438288469
- link link1: mass 1.6995420074353 -> 1.8899542899265
- link link2: mass 0.520903374191751 -> 0.465775740431193
- link link3: mass 0.641519992827807 -> 0.63757668613832
- link link4: mass 0.139838260043534 -> 0.131998325592955
- link link5: mass 0.121592498566107 -> 0.120245289388468
- link link6: mass 0.0556435802970596 -> 0.0892340388435486
- link link7: mass 0.0835736714686863 -> 0.054803438385904
- link link8: mass 0.0680447133767066 -> 0.0245667847957228
Joints:
- joint joint1: axis 0 0 -1 -> 0 0 1; limit lower=0 upper=0.48 effort=0 velocity=0.2 -> lower=0 upper=0.485 effort=0 velocity=0.2; origin xyz=0.27932 -0.673 0.43447 rpy=3.1416 0 0 -> xyz=0.069945 -0.51446 0.1115 rpy=0 0 0
- joint joint2: limit lower=0 upper=0.42 effort=0 velocity=0.2 -> lower=0 upper=0.36 effort=0 velocity=0.2; origin xyz=-0.05665 -0.3632 0.301 rpy=-1.5708 0 0 -> xyz=0 0 0 rpy=-1.5708 0 0
- joint joint3: limit lower=0 upper=0.35 effort=0 velocity=0.2 -> lower=0 upper=0.315 effort=0 velocity=0.15; origin xyz=-0.004 0.056 0.38895 rpy=-3.1416 0 -1.5708 -> xyz=0 0 0 rpy=3.1416 0 0
- joint joint4: axis 1 0 0 -> 0 0 1; limit lower=0 upper=0.2 effort=0 velocity=0.15 -> lower=0 upper=0.185 effort=0 velocity=0.15; origin xyz=-0.007 0.04395 -0.0605 rpy=1.5708 0 1.5708 -> xyz=0 0 0 rpy=0 1.5708 0
- joint joint5: origin xyz=0 -0.048 -0.0285 rpy=1.5708 -1.5708 0 -> xyz=0.80725 0.22497 -0.17472 rpy=0 1.5708 0
- joint joint6: origin xyz=-0.068 0 0.029 rpy=1.5708 0 -1.5708 -> xyz=0 0.068 0.029 rpy=-1.5708 0 0
- joint joint7: origin xyz=0.061 0 0.054 rpy=0 1.5708 0 -> xyz=0.07 0 0.054 rpy=1.5708 0 -1.5708
- joint joint8: axis 0 0 -1 -> 0 0 1; origin xyz=-0.049 0.0018959 -0.061026 rpy=3.1416 1.5708 0 -> xyz=0.0018959 0.049 0.069974 rpy=1.5708 -1.5708 0

Commit message: 0

File: description/urdf/description.urdf (robot description, URDF)
Before this commit: robot engineer2023, 9 links, 8 joints
Links:
- link base_link: mass 5.36255438288469 -> 3.93247154506623
- link link1: mass 1.8899542899265 -> 2.34054483752411
- link link2: mass 0.465775740431193 -> 0.60180055211582
- link link3: mass 0.63757668613832 -> 0.655582856876397
- link link4: mass 0.131998325592955 -> 0.126669555017613
- link link6: mass 0.0892340388435486 -> 0.104211436138975
- link link7: mass 0.054803438385904 -> 0.176077223035249
- link link8: mass 0.0245667847957228 -> 3.28857056779525
Joints:
- joint joint1: limit lower=0 upper=0.485 effort=0 velocity=0.2 -> lower=0 upper=0.48 effort=0 velocity=0.2; origin xyz=0.069945 -0.51446 0.1115 rpy=0 0 0 -> xyz=0.069945 -0.51446 0.1115 rpy=0 0 3.1416
- joint joint2: limit lower=0 upper=0.36 effort=0 velocity=0.2 -> lower=0 upper=0.35 effort=0 velocity=0.15; origin xyz=0 0 0 rpy=-1.5708 0 0 -> xyz=0 0 0 rpy=1.5708 0 0
- joint joint3: origin xyz=0 0 0 rpy=3.1416 0 0 -> xyz=0 0 0 rpy=3.1416 0 3.1416
- joint joint4: limit lower=0 upper=0.185 effort=0 velocity=0.15 -> lower=0 upper=0.185 effort=0 velocity=0.1
- joint joint5: origin xyz=0.80725 0.22497 -0.17472 rpy=0 1.5708 0 -> xyz=0.80725 0.23016 -0.15522 rpy=0 1.5708 0
- joint joint7: axis 0 0 1 -> 0 0 -1; origin xyz=0.07 0 0.054 rpy=1.5708 0 -1.5708 -> xyz=0.07 0 0.054 rpy=1.5708 0 1.5708
- joint joint8: origin xyz=0.0018959 0.049 0.069974 rpy=1.5708 -1.5708 0 -> xyz=-0.022609 0.16849 -0.071802 rpy=1.5658 1.5708 3.1357
